File: source/list-tap.kicad_sch (KiCad schematic)
At the start: 0 parts

Commit message: schematics done awaiting revision
Parts:
- added B1, B2: PESD5V5C1BLYL(TP), list-tap:PESD5V5C1BLYL, symbol list-tap:PESD5V5C1BLYL
- added C1, C12, C14, C15, C16, C2, C5, C7, C8: 100n 50V, list-tap:CAPC1005X04L, symbol list-tap:C0402
- added C10, C11: 22u 10V, list-tap:CAPC1005X04L, symbol list-tap:C0402
- added C13, C6: 10u 10V, list-tap:CAPC1005X04L, symbol list-tap:C0402
- added C3, C4: TBD, list-tap:CAPC1005X04L, symbol list-tap:C0402
- added C9: 10u 25V, list-tap:CAPC1608X06L, symbol list-tap:C0603
- added D1: YLED0402B, list-tap:LED_0402_BLUE, symbol list-tap:LED_0402_BLUE
- added D2: YLED0402R, list-tap:LED_0402_RED, symbol list-tap:LED_0402_RED
- added D3: GREEN, list-tap:LED_0402_GREEN, symbol list-tap:LED_0402_GREEN
- added FB1: BLM18PG121SN1D, list-tap:FB_0603, symbol list-tap:FB_0603
- added J1: TYPE-C-31-M-12, list-tap:HRO_TYPE-C-31-M-12, symbol list-tap:TYPE-C-31-M-12
- added J2: PM2.54-1x4PZZ-H5.7, list-tap:SAMESKY_SSK02-FPH-254-A4, symbol list-tap:PM2.54-1x4PZZ-H5.7
- added L1: 470n 5.3A, CVH252009-1R5M:INDC2520X100N, symbol list-tap:YSMC252008H-R47MB
- added P1: S2B-PH-SM4-TB(LF)(SN), list-tap:JST_S2B-PH-SM4-TB, symbol list-tap:S2B-PH-SM4-TB(LF)(SN)
- added Q1: FS8205A, list-tap:SOP65P640X120-8N, symbol list-tap:FS8205A
- added R1, R2: 5k1, list-tap:RESC1005X04L, symbol list-tap:R0402
- added R10: 100R, list-tap:RESC1005X04L, symbol list-tap:R0402
- added R11, R24, R5, R6: 1k, list-tap:RESC1005X04L, symbol list-tap:R0402
- added R12, R14, R9: 100k, list-tap:RESC1005X04L, symbol list-tap:R0402
- added R13: 150k, list-tap:RESC1005X04L, symbol list-tap:R0402
- added R15: 511k, list-tap:RESC1005X04L, symbol list-tap:R0402
- added R16: 91k, list-tap:RESC1005X04L, symbol list-tap:R0402
- added R17: 34k, list-tap:RESC1005X04L, symbol list-tap:R0402
- added R18: 12k, list-tap:RESC1005X04L, symbol list-tap:R0402
- added R19, R20, R21, R22, R23, R8: 10k, list-tap:RESC1005X04L, symbol list-tap:R0402
- added R25, R26: 4k7, list-tap:RESC1005X04L, symbol list-tap:R0402
- added R3, R4: 22R, list-tap:RESC1005X04L, symbol list-tap:R0402
- added R7: 2k, list-tap:RESC1005X04L, symbol list-tap:R0402
- added SW1, SW2: SKRKAEE020, list-tap:SW2_SKRKAEE020_ALPS, symbol list-tap:SKRKAEE020
- added SW3: PTS815 SJM 250 SMTR LFS, PTS815, symbol list-tap:PTS815-SJM-250-SMTR-LFS
- added TP1, TP2, TP3, TP4, TP5, TP6, TP7: Test Point, list-tap:TP_SMD_D1.5mm, symbol list-tap:TP_SMD_Ø1.5MM
- added U1: DW01A, list-tap:SOT95P280X145-6N, symbol list-tap:DW01A
- added U2: TP4056-42-ESOP8, list-tap:SOP127P600X175-9N, symbol list-tap:TP4056-42-ESOP8
- added U3: USBLC6-2SC6Y, list-tap:SOT23-6L_STM, symbol list-tap:USBLC6-2SC6Y
- added U4: TPS2116DRLR, list-tap:SOTFL50P160X60-8N, symbol list-tap:TPS2116DRLR
- added U5: TPS63805YFFR, list-tap:BGA15N40P5X3_225X134X62N, symbol list-tap:TPS63805YFFR
- added U6: ESP32-C3-WROOM-02-N4, list-tap:MODULE_ESP32-C3-WROOM-02-H4, symbol list-tap:ESP32-C3-WROOM-02-N4
Connections:
- new net: L1.2, U5.B2 (L1), U5.B3 (L1)
- new net: L1.1, U5.D2 (L2), U5.D3 (L2)
- new net: Q1.1, Q1.8
- new net: Q1.4, U1.1 (OD)
- new net: Q1.5, U1.3 (OC)
- new net: D1.K, R5.2
- new net: J1.A5 (CC1), R1.1
- new net: D2.K, R6.2
- new net: C7.1, R10.2, U1.5 (VCC)
- new net: D3.A, R24.1
- new net: R11.2, U1.2 (CS)
- new net: J1.B5 (CC2), R2.1
- new net +3V3: C11.1, C12.1, C13.2, C14.2, J2.2, R14.2, R15.2, R19.2, R20.2, R21.2, R22.2, R23.2, R25.2, R26.2, TP3.1, U5.E2 (VOUT), U5.E3 (VOUT), U6.1 (3V3)
- new net BAT-: Q1.6, Q1.7, R11.1
- new net GND: B1.1 (K1), B2.1 (K1), C1.1, C10.1, C11.2, C12.2, C13.1, C14.1, C15.1, C16.1, C2.1, C3.2, C4.1, C5.2, C6.1, C7.2, C8.1, C9.2, D3.K, J1.A1B12 (GND), J1.B1A12 (GND), J1.SH, J2.1, P1.1, Q1.2, Q1.3, R1.2, R13.1, R16.1, R18.1, R2.2, R7.1, R8.1, R9.2, SW1.2, SW2.2, SW3.4, TP5.1, U1.6 (GND), U2.3 (GND), U2.9 (EP), U3.2 (GND), U4.1 (GND), U5.C1 (AGND), U5.C2 (GND), U5.C3 (GND), U6.19 (GND), U6.20 (GND), U6.21 (GND), U6.22 (GND), U6.23 (GND), U6.24 (GND), U6.25 (GND), U6.26 (GND), U6.27 (GND), U6.28 (GND), U6.29 (GND), U6.30 (GND), U6.31 (GND), U6.32 (GND), U6.33 (GND), U6.34 (GND), U6.35 (GND), U6.36 (GND), U6.37 (GND), U6.38 (GND), U6.39 (GND), U6.9 (GND)
- new net VBAT: B2.2 (K2), C6.2, C9.1, P1.2, R10.1, R17.2, TP2.1, U2.5 (BAT), U4.6 (VIN2)
- new net VBUS: B1.2 (K2), C1.2, FB1.1, J1.A4B9 (VBUS), J1.B4A9 (VBUS)
- new net VIN: C10.2, TP4.1, U4.2 (VOUT), U4.7 (VOUT), U5.A1 (EN), U5.A2 (VIN), U5.A3 (VIN), U5.B1 (MODE)
- new net VUSB: C2.2, C5.1, D1.A, D2.A, FB1.2, R12.2, R9.1, TP1.1, U2.4 (VCC), U2.8 (CE), U3.5 (VBUS), U4.3 (VIN1), U4.5 (MODE)
- new net _usb-n: C3.1, J1.A7 (DN1), J1.B7 (DN2), R3.1, U3.4 (I/O2)
- new net _usb-p: C4.2, J1.A6 (DP1), J1.B6 (DP2), R4.1, U3.1 (I/O1)
- new net boot_n: R21.1, SW1.1, TP6.1, U6.8 (IO9)
- new net btn_n: C16.2, R23.1, SW3.1, U6.17 (IO1)
- new net chrg: R5.1, U2.7 (~{CHRG})
- new net en: R22.1, SW2.1, TP7.1, U6.2 (EN)
- new net io2_strap: R19.1, U6.16 (IO2)
- new net io8_strap: R20.1, U6.7 (IO8)
- new net led: R24.2, U6.15 (IO3)
- new net oled_scl: J2.3, R26.1, U6.6 (IO7)
- new net oled_sda: J2.4, R25.1, U6.5 (IO6)
- new net prog: R7.2, U2.2 (PROG)
- new net stdby: R6.1, U2.6 (~{STDBY})
- new net temp: R8.2, U2.1 (TEMP)
- new net tp_fb: R15.1, R16.2, U5.D1 (FB)
- new net tp_pg: R14.1, U5.E1 (PG)
- new net usb-n: R3.2, U6.13 (IO18)
- new net usb-p: R4.2, U6.14 (IO19)
- new net usb_present: C8.2, R12.1, R13.2, U6.4 (IO5)
- new net vbat_sense: C15.2, R17.1, R18.2, U6.18 (IO0)
- no-connect marks 0 -> 13
Other:
- note added: "3V3 BUCK-BOOST"
- note added: "BATTERY CHARGING AND PROTECTION"
- note added: "BATTERY POWER"
- note added: "BUTTONS"
- note added: "MCU"
- note added: "OLED"
- note added: "POWER MUX"
- note added: "USB POWER & COMMUNICATION"
- title: (none) -> list-tap

Commit message: r2 changes
Parts:
- removed R7: 2k, list-tap:RESC1005X04L, symbol list-tap:R0402
- added R27: 5k, list-tap:RESC1005X04L, symbol list-tap:R0402
- added R28: 10k, list-tap:RESC1005X04L, symbol list-tap:R0402
- added R29: 100k, list-tap:RESC1005X04L, symbol list-tap:R0402
- added R30: 150k, list-tap:RESC1005X04L, symbol list-tap:R0402
- C12: now in the parts list
- C7: value 100n 50V -> 1u 16V; LCSC Part # C53084453 -> C29266; Manufacturer Part Number CC0402X7R50V104MN -> CL05A105KO5NNNC
- R17: value 34k -> 300k; LCSC Part # C843901 -> C2929999; Manufacturer Part Number CRCW040234K0FKED -> FRC0402F3003TS
- R18: value 12k -> 120k; LCSC Part # C2909316 -> C2909314; Manufacturer Part Number FRC0402F1202TS -> FRC0402F1203TS
Connections:
- net +3V3: now also R28.2
- net BAT-: now also C7.2, U1.6 (GND); no longer R11.1
- net GND: now also R11.1, R27.1, R30.1; no longer C7.2, U1.6 (GND)
- net VUSB: now also R29.2
- net prog: now also R27.2
- net tp_st: now reaches U6.3 (IO4)
- net tp_st: now also U4.8 (ST), R28.1
- net tp_pr1: now reaches U4.4 (PR1)
- net tp_pr1: now also R29.1, R30.2
- no-connect marks 13 -> 10
