File: source/v1/list-tap.kicad_sch (KiCad schematic)
At the start: 72 parts, among them J1 TYPE-C-31-M-12, J2 PM2.54-1x4PZZ-H5.7, P1 S2B-PH-SM4-TB(LF)(SN), Q1 FS8205A, SW1 SKRKAEE020, SW2 SKRKAEE020, SW3 PTS815 SJM 250 SMTR LFS, U1 DW01A, U2 TP4056-42-ESOP8, U3 USBLC6-2SC6Y, U4 TPS2116DRLR, U5 TPS63805YFFR, U6 ESP32-C3-WROOM-02-N4

Commit message: layout r1
Parts:
- L1: footprint CVH252009-1R5M:INDC2520X100N -> list-tap:INDC2520X100N
- R17: value 300k -> 340k; LCSC Part # C2929999 -> C2933090; Manufacturer Part Number FRC0402F3003TS -> FRC0402F3403TS
- SW3: footprint PTS815 -> list-tap:PTS815
Connections:
- net BAT-: now also P1.1
- net GND: no longer P1.1
Other:
- moved on the sheet: P1
Changed lines of the file:
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@@
 		)
 	)
-	(text_box "VBAT MAX = 3.7V\n\nESP32 VREF = 1.1V\n\nVADC_MAX = (120k/(120k + 300k)) x 3.7V = 1.0571V"
+	(text_box "VBAT MAX = 4.2V\n\nESP32 VREF = 1.1V\n\nVADC_MAX = (120k/(120k + 340k)) x 4.2V = 1.096V"
 		(exclude_from_sim no)
 		(at 143.51 229.87 0)
-		(size 55.88 14.1714)
+		(size 55.88 12.7)
 		(margins 0.9525 0.9525 0.9525 0.9525)
 		(stroke
@@
 	)
 	(junction
-		(at 72.39 219.71)
-		(diameter 0)
-		(color 0 0 0 0)
-	)
-	(junction
 		(at 485.14 147.32)
 		(diameter 0)
@@
 	)
 	(junction
+		(at 72.39 219.71)
+		(diameter 0)
+		(color 0 0 0 0)
+	)
+	(junction
 		(at 86.36 219.71)
 		(diameter 0)
@@
 	(wire
 		(pts
-			(xy 62.23 222.25) (xy 67.31 222.25)
+			(xy 54.61 222.25) (xy 59.69 222.25)
 		)
 		(stroke
@@
 	(wire
 		(pts
-			(xy 72.39 219.71) (xy 62.23 219.71)
+			(xy 72.39 219.71) (xy 54.61 219.71)
 		)
 		(stroke
@@
 			)
 		)
-		(property "Value" "300k"
+		(property "Value" "340k"
 			(at 116.586 230.378 90)
 			(show_name no)
@@
 			)
 		)
-		(property "Manufacturer Part Number" "FRC0402F3003TS"
+		(property "Manufacturer Part Number" "FRC0402F3403TS"
 			(at 105.41 228.6 0)
 			(hide yes)
@@
 			)
 		)
-		(property "LCSC Part #" "C2929999"
+		(property "LCSC Part #" "C2933090"
 			(at 111.76 227.33 0)
 			(hide yes)
@@
 	)
 	(symbol
+		(lib_id "power:GNDD")
+		(at 59.69 222.25 90)
+		(unit 1)
+		(body_style 1)
+		(exclude_from_sim no)
+		(in_bom yes)
+		(on_board yes)
+		(in_pos_files yes)
+		(dnp no)
+		(fields_autoplaced yes)
+		(property "Reference" "#PWR067"
+			(at 66.04 222.25 0)
+			(hide yes)
+			(show_name no)
+			(do_not_autoplace no)
+			(effects
+				(font
+					(size 1.27 1.27)
+				)
+			)
+		)
+		(property "Value" "BAT-"
+			(at 63.5 222.2499 90)
+			(show_name no)
+			(do_not_autoplace no)
+			(effects
+				(font
+					(size 1.27 1.27)
+				)
+				(justify right)
+			)
+		)
+		(property "Footprint" ""
+			(at 59.69 222.25 0)
+			(hide yes)
+			(show_name no)
+			(do_not_autoplace no)
+			(effects
+				(font
+					(size 1.27 1.27)
+				)
+			)
+		)
+		(property "Datasheet" ""
+			(at 59.69 222.25 0)
+			(hide yes)
+			(show_name no)
+			(do_not_autoplace no)
+			(effects
+				(font
+					(size 1.27 1.27)
+				)
+			)
+		)
+		(property "Description" "Power symbol creates a global label with name \"GNDD\" , digital ground"
+			(at 59.69 222.25 0)
+			(hide yes)
+			(show_name no)
+			(do_not_autoplace no)
+			(effects
+				(font
+					(size 1.27 1.27)
+				)
+			)
+		)
+		(pin "1"
+		)
+		(instances
+			(project "list-tap"
+				(path "/9a2cc030-87ff-40fd-b779-afacc0376da8"
+					(reference "#PWR067")
+					(unit 1)
+				)
+			)
+		)
+	)
+	(symbol
 		(lib_id "power:+2V5")
 		(at 553.72 140.97 0)
@@
 	(symbol
 		(lib_id "list-tap:S2B-PH-SM4-TB(LF)(SN)")
-		(at 57.15 220.98 180)
+		(at 49.53 220.98 180)
 		(unit 1)
 		(body_style 1)
@@
 		(dnp no)
 		(property "Reference" "P1"
-			(at 55.88 214.884 0)
+			(at 48.26 214.884 0)
 			(show_name no)
 			(do_not_autoplace no)
@@
 		)
 		(property "Value" "S2B-PH-SM4-TB(LF)(SN)"
-			(at 57.15 229.362 0)
+			(at 49.53 229.362 0)
 			(show_name no)
 			(do_not_autoplace no)
@@
 		)
 		(property "Footprint" "list-tap:JST_S2B-PH-SM4-TB"
-			(at 57.15 220.98 0)
+			(at 49.53 220.98 0)
 			(hide yes)
 			(show_name no)
@@
 		)
 		(property "Datasheet" ""
-			(at 57.15 220.98 0)
+			(at 49.53 220.98 0)
 			(hide yes)
 			(show_name no)
@@
 		)
 		(property "Description" "Connector Header Surface Mount, Right Angle 2 position 0.079 (2.00mm)"
-			(at 57.15 220.98 0)
+			(at 49.53 220.98 0)
 			(hide yes)
 			(show_name no)
@@
 		)
 		(property "Manufacturer Part Number" "S2B-PH-SM4-TB(LF)(SN)"
-			(at 57.15 220.98 0)
+			(at 49.53 220.98 0)
 			(hide yes)
 			(show_name no)
@@
 		)
 		(property "LCSC Part #" "C295747"
-			(at 57.15 220.98 0)
+			(at 49.53 220.98 0)
 			(hide yes)
 			(show_name no)
@@
 			)
 		)
-		(property "Footprint" "PTS815"
+		(property "Footprint" "list-tap:PTS815"
 			(at 665.48 200.66 0)
 			(hide yes)
@@
 	)
 	(symbol
-		(lib_id "power:GND")
-		(at 67.31 222.25 90)
-		(unit 1)
-		(body_style 1)
-		(exclude_from_sim no)
-		(in_bom yes)
-		(on_board yes)
-		(in_pos_files yes)
-		(dnp no)
-		(fields_autoplaced yes)
-		(property "Reference" "#PWR033"
-			(at 73.66 222.25 0)
-			(hide yes)
-			(show_name no)
-			(do_not_autoplace no)
-			(effects
-				(font
-					(size 1.27 1.27)
-				)
-			)
-		)
-		(property "Value" "GND"
-			(at 71.12 222.2499 90)
-			(hide yes)
-			(show_name no)
-			(do_not_autoplace no)
-			(effects
-				(font
-					(size 1.27 1.27)
-				)
-				(justify right)
-			)
-		)
-		(property "Footprint" ""
-			(at 67.31 222.25 0)
-			(hide yes)
-			(show_name no)
-			(do_not_autoplace no)
-			(effects
-				(font
-					(size 1.27 1.27)
-				)
-			)
-		)
-		(property "Datasheet" ""
-			(at 67.31 222.25 0)
-			(hide yes)
-			(show_name no)
-			(do_not_autoplace no)
-			(effects
-				(font
-					(size 1.27 1.27)
-				)
-			)
-		)
-		(property "Description" "Power symbol creates a global label with name \"GND\" , ground"
-			(at 67.31 222.25 0)
-			(hide yes)
-			(show_name no)
-			(do_not_autoplace no)
-			(effects
-				(font
-					(size 1.27 1.27)
-				)
-			)
-		)
-		(pin "1"
-		)
-		(instances
-			(project "list-tap"
-				(path "/9a2cc030-87ff-40fd-b779-afacc0376da8"
-					(reference "#PWR033")
-					(unit 1)
-				)
-			)
-		)
-	)
-	(symbol
 		(lib_id "list-tap:LED_0402_RED")
 		(at 345.44 80.01 180)
@@
 			)
 		)
-		(property "Footprint" "CVH252009-1R5M:INDC2520X100N"
+		(property "Footprint" "list-tap:INDC2520X100N"
 			(at 416.56 158.75 0)
 			(hide yes)
