File: source/v2/list-tap.kicad_sch (KiCad schematic)
At the start: 59 parts, among them J1 TYPE-C-31-M-12, SW1 SKRKAEE020, SW2 SKRKAEE020, SW3 PTS815 SJM 250 SMTR LFS, U1 DM-OLED096-636, U3 USBLC6-2SC6Y, U4 TPS2116DRLR, U5 TPS63805YFFR, U6 ESP32-C3-WROOM-02-N4

Commit message: bom r2
Parts:
- U1: value DM-OLED096-636 -> PM2.54-1x4PZZ-H5.7; LCSC Part # (none) -> C55218874; Manufacturer Part Number DM-OLED096-636 -> PM2.54-1x4PZZ-H5.7

Commit message: layout r3
Parts:
- removed C12: 100n 50V, list-tap:CAPC1005X04L, symbol list-tap:C0402
- removed R25, R26: 4k7, list-tap:RESC1005X04L, symbol list-tap:R0402
- removed U1: PM2.54-1x4PZZ-H5.7, list-tap:MODULE_DM-OLED096-636, symbol list-tap:DM-OLED096-636
Other:
- note removed: "OLED"
- moved on the sheet: H1, H2, H3, H4

Commit message: layout and routing r4
Connections:
- net GND: now also J1.S1, J1.S2, J1.S3, J1.S4; no longer J1.SH
- net tp_l1: now reaches L1.2, U5.B2 (L1), U5.B3 (L1)
- net tp_l2: now reaches L1.1, U5.D2 (L2), U5.D3 (L2)
- net _usb-n renamed _usb-
- net _usb-p renamed _usb+
- net usb-n renamed usb-
- net usb-p renamed usb+
Other:
- moved on the sheet: L1
Changed lines of the file:
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@@
 	)
 	(junction
+		(at 45.72 110.49)
+		(diameter 0)
+		(color 0 0 0 0)
+	)
+	(junction
 		(at 74.93 80.01)
 		(diameter 0)
@@
 	)
 	(junction
+		(at 45.72 105.41)
+		(diameter 0)
+		(color 0 0 0 0)
+	)
+	(junction
 		(at 172.72 69.85)
 		(diameter 0)
@@
 	)
 	(junction
+		(at 45.72 100.33)
+		(diameter 0)
+		(color 0 0 0 0)
+	)
+	(junction
 		(at 327.66 64.77)
 		(diameter 0)
@@
 	(wire
 		(pts
+			(xy 45.72 100.33) (xy 45.72 105.41)
+		)
+		(stroke
+			(width 0)
+			(type default)
+		)
+	)
+	(wire
+		(pts
 			(xy 448.31 173.99) (xy 453.39 173.99)
 		)
@@
 	(wire
 		(pts
+			(xy 49.53 95.25) (xy 45.72 95.25)
+		)
+		(stroke
+			(width 0)
+			(type default)
+		)
+	)
+	(wire
+		(pts
 			(xy 300.99 243.84) (xy 300.99 248.92)
 		)
@@
 	(wire
 		(pts
+			(xy 45.72 105.41) (xy 49.53 105.41)
+		)
+		(stroke
+			(width 0)
+			(type default)
+		)
+	)
+	(wire
+		(pts
 			(xy 279.4 74.93) (xy 293.37 74.93)
 		)
@@
 	(wire
 		(pts
+			(xy 45.72 100.33) (xy 49.53 100.33)
+		)
+		(stroke
+			(width 0)
+			(type default)
+		)
+	)
+	(wire
+		(pts
 			(xy 453.39 233.68) (xy 459.74 233.68)
 		)
@@
 	(wire
 		(pts
-			(xy 43.18 107.95) (xy 49.53 107.95)
+			(xy 43.18 110.49) (xy 45.72 110.49)
 		)
 		(stroke
@@
 	(wire
 		(pts
-			(xy 285.75 166.37) (xy 275.59 166.37)
+			(xy 279.4 166.37) (xy 275.59 166.37)
 		)
 		(stroke
@@
 	(wire
 		(pts
-			(xy 300.99 166.37) (xy 304.8 166.37)
+			(xy 294.64 166.37) (xy 304.8 166.37)
 		)
 		(stroke
@@
 	(wire
 		(pts
+			(xy 45.72 105.41) (xy 45.72 110.49)
+		)
+		(stroke
+			(width 0)
+			(type default)
+		)
+	)
+	(wire
+		(pts
+			(xy 45.72 110.49) (xy 49.53 110.49)
+		)
+		(stroke
+			(width 0)
+			(type default)
+		)
+	)
+	(wire
+		(pts
+			(xy 45.72 95.25) (xy 45.72 100.33)
+		)
+		(stroke
+			(width 0)
+			(type default)
+		)
+	)
+	(wire
+		(pts
 			(xy 72.39 72.39) (xy 82.55 72.39)
 		)
@@
 		)
 	)
-	(label "_usb-n"
+	(label "_usb-"
 		(at 92.71 151.13 180)
 		(effects
@@
 		)
 	)
-	(label "usb-n"
+	(label "usb-"
 		(at 190.5 147.32 180)
 		(effects
@@
 		)
 	)
-	(label "_usb-n"
+	(label "_usb-"
 		(at 132.08 147.32 0)
 		(effects
@@
 		)
 	)
-	(label "_usb-n"
+	(label "_usb-"
 		(at 83.82 80.01 180)
 		(effects
@@
 		)
 	)
-	(label "usb-p"
+	(label "usb+"
 		(at 542.29 83.82 180)
 		(effects
@@
 		)
 	)
-	(label "usb-n"
+	(label "usb-"
 		(at 542.29 86.36 180)
 		(effects
@@
 		)
 	)
-	(label "_usb-p"
+	(label "_usb+"
 		(at 132.08 160.02 0)
 		(effects
@@
 		)
 	)
+	(label "tp_l2"
+		(at 297.18 173.99 0)
+		(effects
+			(font
+				(size 1.27 1.27)
+			)
+			(justify left bottom)
+		)
+	)
 	(label "en"
 		(at 482.6 76.2 0)
@@
 		)
 	)
-	(label "_usb-p"
+	(label "_usb+"
 		(at 83.82 85.09 180)
 		(effects
@@
 		)
 	)
-	(label "usb-p"
+	(label "usb+"
 		(at 190.5 160.02 180)
 		(effects
@@
 		)
 	)
-	(label "_usb-p"
+	(label "_usb+"
 		(at 29.21 151.13 0)
 		(effects
@@
 		)
 	)
+	(label "tp_l1"
+		(at 297.18 166.37 0)
+		(effects
+			(font
+				(size 1.27 1.27)
+			)
+			(justify left bottom)
+		)
+	)
 	(symbol
 		(lib_id "power:GND")
@@
 			)
 		)
-		(property "Field6" ""
-			(at 59.69 90.17 0)
-			(hide yes)
-			(show_name no)
-			(do_not_autoplace no)
-			(effects
-				(font
-					(size 1.27 1.27)
-				)
-			)
-		)
-		(pin "SH"
+		(pin "S1"
 		)
 		(pin "B7"
@@
 		(pin "A8"
 		)
+		(pin "S3"
+		)
+		(pin "S2"
+		)
+		(pin "S4"
+		)
 		(instances
 			(project "list-tap"
@@
 	(symbol
 		(lib_id "power:GND")
-		(at 43.18 107.95 270)
+		(at 43.18 110.49 270)
 		(unit 1)
 		(body_style 1)
@@
 		(fields_autoplaced yes)
 		(property "Reference" "#PWR03"
-			(at 36.83 107.95 0)
+			(at 36.83 110.49 0)
 			(hide yes)
 			(show_name no)
@@
 		)
 		(property "Value" "GND"
-			(at 39.37 107.9501 90)
+			(at 39.37 110.4901 90)
 			(hide yes)
 			(show_name no)
@@
 		)
 		(property "Footprint" ""
-			(at 43.18 107.95 0)
+			(at 43.18 110.49 0)
 			(hide yes)
 			(show_name no)
@@
 		)
 		(property "Datasheet" ""
-			(at 43.18 107.95 0)
+			(at 43.18 110.49 0)
 			(hide yes)
 			(show_name no)
@@
 		)
 		(property "Description" "Power symbol creates a global label with name \"GND\" , ground"
-			(at 43.18 107.95 0)
+			(at 43.18 110.49 0)
 			(hide yes)
 			(show_name no)
@@
 	(symbol
 		(lib_id "list-tap:YSMC252008H-R47MB")
-		(at 293.37 166.37 0)
+		(at 287.02 166.37 0)
 		(unit 1)
 		(body_style 1)
@@
 		(dnp no)
 		(property "Reference" "L1"
-			(at 293.37 163.322 0)
+			(at 287.02 163.322 0)
 			(show_name no)
 			(do_not_autoplace no)
@@
 		)
 		(property "Value" "470n 5.3A"
-			(at 293.37 168.402 0)
+			(at 287.02 168.402 0)
 			(show_name no)
 			(do_not_autoplace no)
@@
 		)
 		(property "Footprint" "list-tap:INDC2520X100N"
-			(at 293.37 166.37 0)
+			(at 287.02 166.37 0)
 			(hide yes)
 			(show_name no)
@@
 		)
 		(property "Datasheet" ""
-			(at 293.37 166.37 0)
+			(at 287.02 166.37 0)
 			(hide yes)
 			(show_name no)
@@
 		)
 		(property "Description" "Inductors, Fixed, 1.5uH 1MHz 20% | Bourns CVH252009-1R5M"
-			(at 293.37 166.37 0)
+			(at 287.02 166.37 0)
 			(hide yes)
 			(show_name no)
@@
 		)
 		(property "Manufacturer Part Number" "YSMC252008H-R47MB"
-			(at 293.37 166.37 0)
+			(at 287.02 166.37 0)
 			(hide yes)
 			(show_name no)
@@
 		)
 		(property "LCSC Part #" "C46961980"
-			(at 293.37 166.37 0)
+			(at 287.02 166.37 0)
 			(hide yes)
 			(show_name no)
@@
 		)
 		(property "Field6" ""
-			(at 293.37 166.37 0)
+			(at 287.02 166.37 0)
 			(hide yes)
 			(show_name no)
