File: source/v2/list-tap.kicad_pcb (KiCad board)
At the start: 2 copper layers, 37.4 x 55.5 mm, 59 parts, among them J1 TYPE-C-31-M-12, SW1 SKRKAEE020, SW2 SKRKAEE020, SW3 PTS815 SJM 250 SMTR LFS, U1 DM-OLED096-636, U3 USBLC6-2SC6Y, U4 TPS2116DRLR, U5 TPS63805YFFR, U6 ESP32-C3-WROOM-02-N4

Commit message: schematics plot
Parts:
- moved B2 8.48 mm to (134.7, 91.2)
- moved BT1 8.48 mm to (152.5, 89.8)
- moved C9 8.48 mm to (134.7, 88.7)
- moved R17 8.48 mm to (134.9, 86.0)
- moved R18 8.48 mm to (134.9, 84.8)
- moved R29 7.76 mm to (151.7, 88.1), turned to 180 degrees
- moved R30 7.66 mm to (153.8, 88.1), turned to 180 degrees
- moved TP7 6.00 mm to (140.2, 61.4)
- moved L1 5.91 mm to (141.1, 88.1)
- moved R16 5.91 mm to (147.9, 89.2)
- moved C10 5.91 mm to (143.7, 89.2)
- moved C11 5.91 mm to (143.7, 87.0)
- moved R14 5.91 mm to (145.8, 85.1)
- moved R15 5.91 mm to (147.9, 86.7)
- moved TP3 5.91 mm to (143.7, 84.7)
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
Commit message: layout r3
Parts:
- removed C12: 100n 50V, list-tap:CAPC1005X04L
- removed R25, R26: 4k7, list-tap:RESC1005X04L
- removed U1: DM-OLED096-636, list-tap:MODULE_DM-OLED096-636
- moved C16 34.4 mm to (147.5, 73.9)
- moved R23 34.4 mm to (148.8, 73.9)
- moved SW3 34.4 mm to (152.2, 74.5)
- moved R1 19.0 mm to (146.7, 92.7), turned to 90 degrees
- moved J1 17.7 mm to (152.2, 95.1), turned to 0 degrees
- moved TP3 16.7 mm to (158.5, 77.0), turned to 0 degrees
- moved U3 16.3 mm to (146.2, 86.4)
- moved H4 15.3 mm to (137.5, 94.2)
- moved H3 15.3 mm to (167.0, 94.2)
- moved L1 14.7 mm to (152.2, 78.5), turned to 180 degrees
- moved TP4 13.4 mm to (147.4, 80.8)
- moved R2 12.8 mm to (157.9, 92.7), turned to 90 degrees
- moved R28 12.5 mm to (142.0, 81.8)
- moved R29 12.5 mm to (143.9, 78.4)
- moved U4 12.5 mm to (144.2, 80.5)
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Other:
- board size 37.4 x 55.5 mm -> 35 x 40 mm

Commit message: layout and routing r4
Parts:
- moved C8 6.67 mm to (141.6, 63.0)
- moved R18 6.28 mm to (139.2, 76.9), turned to 180 degrees
- moved TP3 4.34 mm to (156.0, 80.5)
- moved R17 3.96 mm to (139.2, 78.1), turned to 0 degrees
- moved R13 2.41 mm to (163.5, 81.1), turned to -90 degrees
- moved TP4 1.60 mm to (148.9, 80.6)
- moved R12 0.94 mm to (163.5, 83.7), turned to -90 degrees
- moved U4 0.68 mm to (143.8, 80.0)
- moved R28 0.68 mm to (141.5, 81.3)
- moved R29 0.68 mm to (143.4, 77.9)
- moved R30 0.68 mm to (145.5, 77.9)
- moved L1 0.57 mm to (152.2, 77.9)
- moved C3 0.26 mm to (151.1, 88.3)
- moved C4 0.26 mm to (153.6, 88.4)
- moved R3 0.26 mm to (151.6, 86.8)
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Connections:
- net /_usb-n renamed /_usb-
- net /_usb-p renamed /_usb+
- net /usb-n renamed /usb-
- net /usb-p renamed /usb+
- net Net-(L1-Pad1) renamed /tp_l2
- net Net-(L1-Pad2) renamed /tp_l1
- J1 pad S1: (no net) -> GND
- J1 pad S2: (no net) -> GND
- J1 pad S3: (no net) -> GND
- J1 pad S4: (no net) -> GND
Routing:
- net /vbat_sense: track 0.00 -> 40.5 mm, vias 0 -> 2
- net /usb_present: track 0.00 -> 35.2 mm, vias 0 -> 2
- net /usb+: track 0.00 -> 30.6 mm, vias 0 -> 2
- net /usb-: track 0.00 -> 29.9 mm, vias 0 -> 2
- net /tp_st: track 0.00 -> 26.4 mm, vias 0 -> 4
- net /btn_n: track 0.00 -> 21.7 mm
- net +3V3: track 0.00 -> 20.1 mm, vias 0 -> 12
- net VUSB: track 0.00 -> 15.9 mm, vias 0 -> 5
- net /led: track 0.00 -> 14.7 mm, vias 0 -> 2
- net /_usb-: track 0.00 -> 14.2 mm, vias 0 -> 2
- net VBUS: track 0.00 -> 14.1 mm, vias 0 -> 2
- net /_usb+: track 0.00 -> 13.6 mm, vias 0 -> 2
- net /en: track 0.00 -> 12.0 mm
- net VBAT: track 0.00 -> 10.7 mm
- net /boot_n: track 0.00 -> 10.3 mm
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- added copper zone on B.Cu, net +3V3
- added copper zone on F.Cu, net /tp_l1
- added copper zone on F.Cu, net /tp_l2
- added copper zone on F.Cu, net GND
- added copper zone on In1.Cu, net GND
- added copper zone on In2.Cu, net GND
- added copper zone on F.Cu, net VSYS
- added copper zone on B.Cu, net VUSB
Other:
- copper layers 2 -> 4

Commit message: layout and routing r4
Routing:
- net GND: vias 28 -> 37
