File: source/v3/list-tap.kicad_sch (KiCad schematic)
At the start: 45 parts, among them J1 HX PH254-01-04-Z-L11.5, J2 HX PH254-01-04-Z-L11.5, SW1 SKRKAEE020, SW2 SKRKAEE020, SW3 PTS815 SJM 250 SMTR LFS, U3 USBLC6-2SC6Y, U5 TPS63805YFFR, U6 ESP32-C3-WROOM-02-N4

Commit message: v3 editions
Parts:
- J2: now not fitted; now left out of the parts list
Connections:
- net oled_scl: no longer names the net of U6.6 (IO7)
- net oled_sda: no longer names the net of U6.5 (IO6)
- no-connect marks 7 -> 9
Changed lines of the file:
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@@
+	)
+	(no_connect
+		(at 391.16 85.09)
 	)
 	(no_connect
@@
 	)
 	(no_connect
+		(at 391.16 82.55)
+	)
+	(no_connect
 		(at 64.77 171.45)
 	)
@@
 	(wire
 		(pts
-			(xy 378.46 82.55) (xy 391.16 82.55)
-		)
-		(stroke
-			(width 0)
-			(type default)
-		)
-	)
-	(wire
-		(pts
 			(xy 163.83 152.4) (xy 172.72 152.4)
 		)
@@
 		(pts
 			(xy 67.31 116.84) (xy 80.01 116.84)
-		)
-		(stroke
-			(width 0)
-			(type default)
-		)
-	)
-	(wire
-		(pts
-			(xy 378.46 85.09) (xy 391.16 85.09)
 		)
 		(stroke
@@
 		)
 	)
-	(label "oled_scl"
-		(at 378.46 85.09 0)
-		(effects
-			(font
-				(size 1.27 1.27)
-			)
-			(justify left bottom)
-		)
-	)
 	(label "en"
 		(at 334.01 232.41 0)
@@
 			)
 			(justify right bottom)
-		)
-	)
-	(label "oled_sda"
-		(at 378.46 82.55 0)
-		(effects
-			(font
-				(size 1.27 1.27)
-			)
-			(justify left bottom)
 		)
 	)
@@
 		(body_style 1)
 		(exclude_from_sim no)
-		(in_bom yes)
+		(in_bom no)
 		(on_board yes)
 		(in_pos_files yes)
-		(dnp no)
+		(dnp yes)
 		(property "Reference" "J2"
 			(at 16.256 102.87 0)

Commit message: fabrication files prepared
Parts:
- L1: LCSC Part # C46961980 -> C5179442; Manufacturer Part Number YSMC252008H-R47MB -> FWP252012P-R47ML
- U3: FT Rotation Offset (none) -> -90
- U6: FT Position Offset (none) -> 0,-3.1
Connections:
- net VUSB is gone; now on net +3V3: U3.5 (VBUS)
- net GND: now also U5.B1 (MODE)
- net VBAT: no longer U5.B1 (MODE)

Commit message: 3v3 zener clamping
Parts:
- added D1, D2: BZT52C3V3S-TP, list-tap:SOD2512X115N, symbol list-tap:BZT52C3V3S-TP
- L1: LCSC Part # C5179442 -> C46961980; Manufacturer Part Number FWP252012P-R47ML -> YSMC252008H-R47MB
- U3: FT Rotation Offset -90 -> (none)
- U6: FT Position Offset 0,-3.1 -> (none)
Connections:
- net +3V3: now also D1.K, D2.K
- net GND: now also D1.A, D2.A
Other:
- moved on the sheet: C18
