File: source/v3/list-tap.kicad_sch (KiCad schematic)
At the start: 47 parts, among them J1 HX PH254-01-04-Z-L11.5, J2 HX PH254-01-04-Z-L11.5, SW1 SKRKAEE020, SW2 SKRKAEE020, SW3 PTS815 SJM 250 SMTR LFS, U3 USBLC6-2SC6Y, U5 TPS63805YFFR, U6 ESP32-C3-WROOM-02-N4

Commit message: L1 swap
Parts:
- L1: value 470n 5.3A -> 470n 5.5A; LCSC Part # C46961980 -> C54557079; Manufacturer Part Number YSMC252008H-R47MB -> PCT252010-R47-M
Changed lines of the file:
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@@
 			)
 		)
-		(property "Value" "470n 5.3A"
+		(property "Value" "470n 5.5A"
 			(at 182.88 167.132 0)
 			(show_name no)
@@
 			)
 		)
-		(property "Manufacturer Part Number" "YSMC252008H-R47MB"
+		(property "Manufacturer Part Number" "PCT252010-R47-M"
 			(at 182.88 165.1 0)
 			(hide yes)
@@
 			)
 		)
-		(property "LCSC Part #" "C46961980"
+		(property "LCSC Part #" "C54557079"
 			(at 182.88 165.1 0)
 			(hide yes)

Commit message: MY-2450-02 battery holder
Parts:
- removed BT1: BC-2007, list-tap:BAT_BC-2007, symbol list-tap:BC-2007
- added BT1: MY-2450-02, list-tap:BAT_BK-880, symbol list-tap:MY-2450-02
- D1, D2: now not fitted
Connections:
- net GND: now also BT1.-
- net VBAT: now also BT1.S+1, BT1.S+2
Changed lines of the file:
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@@
 		(on_board yes)
 		(in_pos_files yes)
-		(dnp no)
+		(dnp yes)
 		(property "Reference" "D1"
 			(at 293.624 60.96 90)
@@
 	)
 	(symbol
+		(lib_id "list-tap:MY-2450-02")
+		(at 201.93 81.28 270)
+		(unit 1)
+		(body_style 1)
+		(exclude_from_sim no)
+		(in_bom yes)
+		(on_board yes)
+		(in_pos_files yes)
+		(dnp no)
+		(fields_autoplaced yes)
+		(property "Reference" "BT1"
+			(at 205.74 79.8829 90)
+			(show_name no)
+			(do_not_autoplace no)
+			(effects
+				(font
+					(size 1.27 1.27)
+				)
+				(justify left)
+			)
+		)
+		(property "Value" "MY-2450-02"
+			(at 205.74 82.4229 90)
+			(show_name no)
+			(do_not_autoplace no)
+			(effects
+				(font
+					(size 1.27 1.27)
+				)
+				(justify left)
+			)
+		)
+		(property "Footprint" "list-tap:BAT_BK-880"
+			(at 201.93 81.28 0)
+			(hide yes)
+			(show_name no)
+			(do_not_autoplace no)
+			(effects
+				(font
+					(size 1.27 1.27)
+				)
+				(justify bottom)
+			)
+		)
+		(property "Datasheet" ""
+			(at 201.93 81.28 0)
+			(hide yes)
+			(show_name no)
+			(do_not_autoplace no)
+			(effects
+				(font
+					(size 1.27 1.27)
+				)
+			)
+		)
+		(property "Description" "coin cell battery holders, cr2450 holder, coin cell retainers"
+			(at 201.93 81.28 0)
+			(hide yes)
+			(show_name no)
+			(do_not_autoplace no)
+			(effects
+				(font
+					(size 1.27 1.27)
+				)
+				(justify bottom)
+			)
+		)
+		(property "Manufacturer Part Number" "MY-2450-02"
+			(at 201.93 81.28 0)
+			(hide yes)
+			(show_name no)
+			(do_not_autoplace no)
+			(effects
+				(font
+					(size 1.27 1.27)
+				)
+			)
+		)
+		(property "LCSC Part #" "C2979177"
+			(at 201.93 81.28 0)
+			(hide yes)
+			(show_name no)
+			(do_not_autoplace no)
+			(effects
+				(font
+					(size 1.27 1.27)
+				)
+			)
+		)
+		(pin "S+2"
+		)
+		(pin "-"
+		)
+		(pin "S+1"
+		)
+		(instances
+			(project "list-tap"
+				(path "/9a2cc030-87ff-40fd-b779-afacc0376da8"
+					(reference "BT1")
+					(unit 1)
+				)
+			)
+		)
+	)
+	(symbol
 		(lib_id "list-tap:R0402")
 		(at 349.25 213.36 90)
@@
 				(path "/9a2cc030-87ff-40fd-b779-afacc0376da8"
 					(reference "#PWR045")
-					(unit 1)
-				)
-			)
-		)
-	)
-	(symbol
-		(lib_id "list-tap:BC-2007")
-		(at 201.93 81.28 270)
-		(unit 1)
-		(body_style 1)
-		(exclude_from_sim no)
-		(in_bom yes)
-		(on_board yes)
-		(in_pos_files yes)
-		(dnp no)
-		(fields_autoplaced yes)
-		(property "Reference" "BT1"
-			(at 205.74 79.8829 90)
-			(show_name no)
-			(do_not_autoplace no)
-			(effects
-				(font
-					(size 1.27 1.27)
-				)
-				(justify left)
-			)
-		)
-		(property "Value" "BC-2007"
-			(at 205.74 82.4229 90)
-			(show_name no)
-			(do_not_autoplace no)
-			(effects
-				(font
-					(size 1.27 1.27)
-				)
-				(justify left)
-			)
-		)
-		(property "Footprint" "list-tap:BAT_BC-2007"
-			(at 201.93 81.28 0)
-			(hide yes)
-			(show_name no)
-			(do_not_autoplace no)
-			(effects
-				(font
-					(size 1.27 1.27)
-				)
-				(justify bottom)
-			)
-		)
-		(property "Datasheet" ""
-			(at 201.93 81.28 0)
-			(hide yes)
-			(show_name no)
-			(do_not_autoplace no)
-			(effects
-				(font
-					(size 1.27 1.27)
-				)
-			)
-		)
-		(property "Description" "coin cell battery holders, cr2450 holder, coin cell retainers"
-			(at 201.93 81.28 0)
-			(hide yes)
-			(show_name no)
-			(do_not_autoplace no)
-			(effects
-				(font
-					(size 1.27 1.27)
-				)
-				(justify bottom)
-			)
-		)
-		(property "Manufacturer Part Number" "BC-2007"
-			(at 201.93 81.28 0)
-			(hide yes)
-			(show_name no)
-			(do_not_autoplace no)
-			(effects
-				(font
-					(size 1.27 1.27)
-				)
-			)
-		)
-		(property "LCSC Part #" "C5556994"
-			(at 201.93 81.28 0)
-			(hide yes)
-			(show_name no)
-			(do_not_autoplace no)
-			(effects
-				(font
-					(size 1.27 1.27)
-				)
-			)
-		)
-		(pin "-"
-		)
-		(pin "S+2"
-		)
-		(pin "S+1"
-		)
-		(instances
-			(project "list-tap"
-				(path "/9a2cc030-87ff-40fd-b779-afacc0376da8"
-					(reference "BT1")
 					(unit 1)
 				)
@@
 		(on_board yes)
 		(in_pos_files yes)
-		(dnp no)
+		(dnp yes)
 		(property "Reference" "D2"
 			(at 38.354 116.078 0)
