File: source/v3/list-tap.kicad_pcb (KiCad board)
At the start: 2 copper layers, 35 x 36 mm, 50 parts, among them J1 HX PH254-01-04-Z-L11.5, J2 HX PH254-01-04-Z-L11.5, SW1 SKRKAEE020, SW2 SKRKAEE020, SW3 PTS815 SJM 250 SMTR LFS, U3 USBLC6-2SC6Y, U5 TPS63805YFFR, U6 ESP32-C3-WROOM-02-N4

Commit message: fabrication files prepared
Parts:
- moved kibuzzard-6AE057E3 1.00 mm to (159.7, 90.4), turned to 90 degrees
Connections:
- U3 pad 5: VUSB -> +3V3
- U5 pad B1: VBAT -> GND
- U6 pad 5: /oled_sda -> unconnected-(U6-IO6-Pad5)
- U6 pad 6: /oled_scl -> unconnected-(U6-IO7-Pad6)
Routing:
- net +3V3: track 24.9 -> 33.7 mm, vias 13 -> 15
- net VUSB: track 1.06 -> 0.00 mm, vias 1 -> 0
- net /boot_n: track 16.4 -> 15.7 mm
Other:
- outline, holes or cut-outs redrawn

Commit message: 3v3 zener clamping
Parts:
- added D1: BZT52C3V3S-TP, list-tap:SOD2512X115N, F.Cu at (166.4, 63.0)
- added D2: BZT52C3V3S-TP, list-tap:SOD2512X115N, F.Cu at (159.5, 90.0)
- moved kibuzzard-6AE057E3 2.63 mm to (162.3, 90.4)
Routing:
- net +3V3: track 33.7 -> 38.7 mm

Commit message: L1 swap
Parts:
- L1: value 470n 5.3A -> 470n 5.5A
Changed lines of the file:
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@@
 			)
 		)
-		(property "Value" "470n 5.3A"
+		(property "Value" "470n 5.5A"
 			(at 1.29 1.7 0)
 			(layer "F.Fab")
@@
 			)
 		)
-		(property "Manufacturer Part Number" "YSMC252008H-R47MB"
+		(property "Manufacturer Part Number" "PCT252010-R47-M"
 			(at 0 0 180)
 			(unlocked yes)
@@
 			)
 		)
-		(property "LCSC Part #" "C46961980"
+		(property "LCSC Part #" "C54557079"
 			(at 0 0 180)
 			(unlocked yes)

Commit message: MY-2450-02 battery holder
Parts:
- BT1: value BC-2007 -> MY-2450-02; footprint list-tap:BAT_BC-2007 -> list-tap:BAT_BK-880
- moved BT1 0.05 mm to (152.2, 73.2)
Routing:
- net GND: track 33.5 -> 23.1 mm
